File: raspberry.sch (KiCad schematic (older format))
At the start: 1 part, among them J2 raspberry

Commit message: Add I2C EEPROM
Parts:
- added C?: C, symbol device:C
- added R? (x2): 3k9, symbol device:R
- added R?: 1k, symbol device:R
- added U?: CAT24C32W, faltom:OnSemi_SOIC8, symbol faltom:CAT24C32W
Connections:
- net labels added: +3V3, GND, pi_eeprom_scl_3v3, pi_eeprom_sda_3v3
- wire segments 0 -> 28
Other:
- note added: "HAT EEPROM"
Changed lines of the file:
@@
 L faltomPi-rescue:raspberry-RESCUE-FaltomPi-FaltomPi-rescue J2
 U 1 1 5516AE26
-P 4700 2700
+P 6500 1500
 AR Path="/5516AE26" Ref="J2"  Part="1"
 AR Path="/5515D395/5516AE26" Ref="J1"  Part="1"
-F 0 "J1" H 5450 2950 60  0000 C CNN
-F 1 "raspberry" H 5450 2850 60  0000 C CNN
-F 2 "faltom:rpi_hat_th" H 4700 2700 60  0001 C CNN
-F 3 "" H 4700 2700 60  0000 C CNN
-	1    4700 2700
+F 0 "J1" H 7250 1750 60  0000 C CNN
+F 1 "raspberry" H 7250 1650 60  0000 C CNN
+F 2 "faltom:rpi_hat_th" H 6500 1500 60  0001 C CNN
+F 3 "" H 6500 1500 60  0000 C CNN
+	1    6500 1500
 	1    0    0    -1
 $EndComp
+$Comp
+L faltom:CAT24C32W U?
+U 1 1 5AAE53A0
+P 1750 2000
+F 0 "U?" H 1850 2250 50  0000 C CNN
+F 1 "CAT24C32W" H 2000 1750 50  0000 C CNN
+F 2 "faltom:OnSemi_SOIC8" H 1750 1750 50  0001 C CNN
+F 3 "https://docs-emea.rs-online.com/webdocs/121e/0900766b8121eacf.pdf" H 1750 1750 50  0001 C CNN
+	1    1750 2000
+	1    0    0    -1
+$EndComp
+$Comp
+L power:GND #PWR?
+U 1 1 5AAE5464
+P 1750 2550
+F 0 "#PWR?" H 1750 2300 50  0001 C CNN
+F 1 "GND" H 1755 2377 50  0000 C CNN
+F 2 "" H 1750 2550 50  0001 C CNN
+F 3 "" H 1750 2550 50  0001 C CNN
+	1    1750 2550
+	1    0    0    -1
+$EndComp
+Wire Wire Line
+	1750 2400 1750 2550
+$Comp
+L power:+3V3 #PWR?
+U 1 1 5AAE55B3
+P 1750 900
+F 0 "#PWR?" H 1750 750 50  0001 C CNN
+F 1 "+3V3" H 1765 1073 50  0000 C CNN
+F 2 "" H 1750 900 50  0001 C CNN
+F 3 "" H 1750 900 50  0001 C CNN
+	1    1750 900
+	1    0    0    -1
+$EndComp
+Wire Wire Line
+	1750 900  1750 1000
+$Comp
+L power:GND #PWR?
+U 1 1 5AAE55D3
+P 1150 2550
+F 0 "#PWR?" H 1150 2300 50  0001 C CNN
+F 1 "GND" H 1155 2377 50  0000 C CNN
+F 2 "" H 1150 2550 50  0001 C CNN
+F 3 "" H 1150 2550 50  0001 C CNN
+	1    1150 2550
+	1    0    0    -1
+$EndComp
+Wire Wire Line
+	1150 2500 1150 2100
+Wire Wire Line
+	1150 1900 1300 1900
+Wire Wire Line
+	1300 2000 1150 2000
+Connection ~ 1150 2000
+Wire Wire Line
+	1150 2000 1150 1900
+Wire Wire Line
+	1300 2100 1150 2100
+Connection ~ 1150 2100
+Wire Wire Line
+	1150 2100 1150 2000
+$Comp
+L device:C C?
+U 1 1 5AAE57B6
+P 2000 1250
+F 0 "C?" H 2115 1296 50  0000 L CNN
+F 1 "C" H 2115 1205 50  0000 L CNN
+F 2 "" H 2038 1100 50  0001 C CNN
+F 3 "" H 2000 1250 50  0001 C CNN
+	1    2000 1250
+	1    0    0    -1
+$EndComp
+$Comp
+L power:GND #PWR?
+U 1 1 5AAE584E
+P 2000 1500
+F 0 "#PWR?" H 2000 1250 50  0001 C CNN
+F 1 "GND" H 2005 1327 50  0000 C CNN
+F 2 "" H 2000 1500 50  0001 C CNN
+F 3 "" H 2000 1500 50  0001 C CNN
+	1    2000 1500
+	1    0    0    -1
+$EndComp
+Wire Wire Line
+	2000 1500 2000 1400
+Wire Wire Line
+	2000 1100 2000 1000
+Wire Wire Line
+	2000 1000 1750 1000
+Connection ~ 1750 1000
+Wire Wire Line
+	1750 1000 1750 1600
+$Comp
+L device:R R?
+U 1 1 5AAE5948
+P 2400 1250
+F 0 "R?" H 2470 1296 50  0000 L CNN
+F 1 "3k9" H 2470 1205 50  0000 L CNN
+F 2 "" V 2330 1250 50  0001 C CNN
+F 3 "" H 2400 1250 50  0001 C CNN
+	1    2400 1250
+	1    0    0    -1
+$EndComp
+$Comp
+L device:R R?
+U 1 1 5AAE5976
+P 2700 1250
+F 0 "R?" H 2770 1296 50  0000 L CNN
+F 1 "3k9" H 2770 1205 50  0000 L CNN
+F 2 "" V 2630 1250 50  0001 C CNN
+F 3 "" H 2700 1250 50  0001 C CNN
+	1    2700 1250
+	1    0    0    -1
+$EndComp
+$Comp
+L device:R R?
+U 1 1 5AAE5998
+P 3000 1250
+F 0 "R?" H 3070 1296 50  0000 L CNN
+F 1 "1k" H 3070 1205 50  0000 L CNN
+F 2 "" V 2930 1250 50  0001 C CNN
+F 3 "" H 3000 1250 50  0001 C CNN
+	1    3000 1250
+	1    0    0    -1
+$EndComp
+Wire Wire Line
+	2000 1000 2400 1000
+Wire Wire Line
+	3000 1000 3000 1100
+Connection ~ 2000 1000
+Wire Wire Line
+	2700 1100 2700 1000
+Connection ~ 2700 1000
+Wire Wire Line
+	2700 1000 3000 1000
+Wire Wire Line
+	2400 1100 2400 1000
+Connection ~ 2400 1000
+Wire Wire Line
+	2400 1000 2700 1000
+Wire Wire Line
+	2400 1400 2400 1900
+Wire Wire Line
+	2400 1900 2200 1900
+Wire Wire Line
+	2700 1400 2700 2000
+Wire Wire Line
+	2700 2000 2200 2000
+Wire Wire Line
+	3000 1400 3000 2100
+Wire Wire Line
+	3000 2100 2200 2100
+Connection ~ 2400 1900
+Connection ~ 2700 2000
+Text Label 3100 1900 0    50   ~ 0
+pi_eeprom_sda_3v3
+Text Label 3100 2000 0    50   ~ 0
+pi_eeprom_scl_3v3
+Wire Wire Line
+	2400 1900 3900 1900
+Wire Wire Line
+	2700 2000 3900 2000
+Wire Notes Line
+	4050 500  4050 2850
+Wire Notes Line
+	4050 2850 500  2850
+Text Notes 500  600  0    50   ~ 0
+HAT EEPROM
+Text Label 8300 2800 0    50   ~ 0
+pi_eeprom_scl_3v3
+Wire Wire Line
+	8200 2800 9050 2800
+Text Label 5450 2800 0    50   ~ 0
+pi_eeprom_sda_3v3
+Wire Wire Line
+	5400 2800 6300 2800
 $EndSCHEMATC

Commit message: Add rasperry supply protection
Parts:
- added R?: 10k, symbol device:R
- added R?: 47k, symbol device:R
- added U?: DMG2305UX, faltom:DiodeInc_SOT-23, symbol faltom:DMG2305UX
- added U?: DMMT5401-7-F, faltom:DiodeInc_SOT-26, symbol faltom:DMMT5401-7-F
Connections:
- net labels added: +5V, pi_pwr_5v
- wire segments 28 -> 51
Other:
- note added: "Pi supply"
Changed lines of the file:
@@
 L faltomPi-rescue:raspberry-RESCUE-FaltomPi-FaltomPi-rescue J2
 U 1 1 5516AE26
-P 6500 1500
+P 4200 4350
 AR Path="/5516AE26" Ref="J2"  Part="1"
 AR Path="/5515D395/5516AE26" Ref="J1"  Part="1"
-F 0 "J1" H 7250 1750 60  0000 C CNN
-F 1 "raspberry" H 7250 1650 60  0000 C CNN
-F 2 "faltom:rpi_hat_th" H 6500 1500 60  0001 C CNN
-F 3 "" H 6500 1500 60  0000 C CNN
-	1    6500 1500
+F 0 "J1" H 4950 4600 60  0000 C CNN
+F 1 "raspberry" H 4950 4500 60  0000 C CNN
+F 2 "faltom:rpi_hat_th" H 4200 4350 60  0001 C CNN
+F 3 "" H 4200 4350 60  0000 C CNN
+	1    4200 4350
 	1    0    0    -1
 $EndComp
@@
 Wire Notes Line
 	4050 500  4050 2850
-Wire Notes Line
-	4050 2850 500  2850
 Text Notes 500  600  0    50   ~ 0
 HAT EEPROM
-Text Label 8300 2800 0    50   ~ 0
+Text Label 6000 5650 0    50   ~ 0
 pi_eeprom_scl_3v3
 Wire Wire Line
-	8200 2800 9050 2800
-Text Label 5450 2800 0    50   ~ 0
+	5900 5650 6750 5650
+Text Label 3150 5650 0    50   ~ 0
 pi_eeprom_sda_3v3
 Wire Wire Line
-	5400 2800 6300 2800
+	3100 5650 4000 5650
+$Comp
+L faltom:DMG2305UX U?
+U 1 1 5AAE8E7C
+P 5750 1050
+F 0 "U?" V 5993 1050 50  0000 C CNN
+F 1 "DMG2305UX" V 5902 1050 50  0000 C CNN
+F 2 "faltom:DiodeInc_SOT-23" H 5750 1050 50  0001 C CNN
+F 3 "https://docs-emea.rs-online.com/webdocs/1332/0900766b81332207.pdf" H 5850 1150 50  0001 C CNN
+	1    5750 1050
+	0    -1   -1   0
+$EndComp
+$Comp
+L faltom:DMMT5401-7-F U?
+U 1 1 5AAE97BF
+P 5750 1600
+F 0 "U?" H 6178 1646 50  0000 L CNN
+F 1 "DMMT5401-7-F" H 6178 1555 50  0000 L CNN
+F 2 "faltom:DiodeInc_SOT-26" H 6450 1950 50  0001 C CNN
+F 3 "https://docs-emea.rs-online.com/webdocs/0e49/0900766b80e49504.pdf" H 6450 1950 50  0001 C CNN
+	1    5750 1600
+	1    0    0    -1
+$EndComp
+$Comp
+L power:+5V #PWR?
+U 1 1 5AAE9AF6
+P 5000 700
+F 0 "#PWR?" H 5000 550 50  0001 C CNN
+F 1 "+5V" H 5015 873 50  0000 C CNN
+F 2 "" H 5000 700 50  0001 C CNN
+F 3 "" H 5000 700 50  0001 C CNN
+	1    5000 700
+	1    0    0    -1
+$EndComp
+Wire Wire Line
+	5000 700  5000 1050
+Wire Wire Line
+	5000 1050 5450 1050
+Wire Wire Line
+	5450 1250 5450 1050
+Connection ~ 5450 1050
+Wire Wire Line
+	5450 1050 5550 1050
+Wire Wire Line
+	6050 1250 6050 1050
+Wire Wire Line
+	6050 1050 6600 1050
+Wire Wire Line
+	6050 1050 5950 1050
+Connection ~ 6050 1050
+$Comp
+L device:R R?
+U 1 1 5AAEA86E
+P 5450 2300
+F 0 "R?" H 5520 2346 50  0000 L CNN
+F 1 "10k" H 5520 2255 50  0000 L CNN
+F 2 "" V 5380 2300 50  0001 C CNN
+F 3 "" H 5450 2300 50  0001 C CNN
+	1    5450 2300
+	1    0    0    -1
+$EndComp
+$Comp
+L power:GND #PWR?
+U 1 1 5AAEA8BC
+P 5450 2550
+F 0 "#PWR?" H 5450 2300 50  0001 C CNN
+F 1 "GND" H 5455 2377 50  0000 C CNN
+F 2 "" H 5450 2550 50  0001 C CNN
+F 3 "" H 5450 2550 50  0001 C CNN
+	1    5450 2550
+	1    0    0    -1
+$EndComp
+$Comp
+L device:R R?
+U 1 1 5AAEA8D9
+P 6050 2300
+F 0 "R?" H 6120 2346 50  0000 L CNN
+F 1 "47k" H 6120 2255 50  0000 L CNN
+F 2 "" V 5980 2300 50  0001 C CNN
+F 3 "" H 6050 2300 50  0001 C CNN
+	1    6050 2300
+	1    0    0    -1
+$EndComp
+$Comp
+L power:GND #PWR?
+U 1 1 5AAEA921
+P 6050 2550
+F 0 "#PWR?" H 6050 2300 50  0001 C CNN
+F 1 "GND" H 6055 2377 50  0000 C CNN
+F 2 "" H 6050 2550 50  0001 C CNN
+F 3 "" H 6050 2550 50  0001 C CNN
+	1    6050 2550
+	1    0    0    -1
+$EndComp
+Wire Wire Line
+	6050 2550 6050 2450
+Wire Wire Line
+	5450 2150 5450 2100
+Wire Wire Line
+	5850 1950 5850 2100
+Wire Wire Line
+	5850 2100 5650 2100
+Connection ~ 5450 2100
+Wire Wire Line
+	5450 2100 5450 1950
+Wire Wire Line
+	5750 1350 5750 2000
+Wire Wire Line
+	5750 2000 6050 2000
+Wire Wire Line
+	6050 2000 6050 1950
+Wire Wire Line
+	6050 2000 6050 2150
+Connection ~ 6050 2000
+Wire Wire Line
+	5650 1950 5650 2100
+Connection ~ 5650 2100
+Wire Wire Line
+	5650 2100 5450 2100
+Wire Wire Line
+	5450 2450 5450 2550
+Text Label 6250 1050 0    50   ~ 0
+pi_pwr_5v
+Text Label 6000 4350 0    50   ~ 0
+pi_pwr_5v
+Wire Wire Line
+	5900 4350 5950 4350
+Wire Wire Line
+	5900 4450 5950 4450
+Wire Wire Line
+	5950 4450 5950 4350
+Connection ~ 5950 4350
+Wire Wire Line
+	5950 4350 6750 4350
+Wire Notes Line
+	7200 2850 7200 500
+Wire Notes Line
+	500  2850 7200 2850
+Text Notes 4100 600  0    50   ~ 0
+Pi supply
 $EndSCHEMATC

Commit message: Add DigitalIO connector
Parts:
- added J?: DigitalIO_OUT, faltom:Molex_43045-1201, symbol faltom:DigitalIO_OUT
- added R? (x3): 10k, symbol device:R
Connections:
- net labels added: int_3v3, latch_3v3, miso_3v3, mosi_3v3, rx_3v3, sck_3v3, set_3v3, tx_3v3
- wire segments 51 -> 103
Other:
- note added: "DigitalIO"
